File: FlightComputerBoardV1/POWER.kicad_sch (KiCad schematic)
At the start: 0 parts

Commit message: buck converter 5v
Parts:
- added C10, C11: 10uF, cappy1:CAP_GRM32_3p5X2p7X2p7_MUR, symbol Device:C
- added C12, C14: 0.1uF, cappy3:CAP_885012206_WRE, symbol Device:C
- added C13: 47nF, cappy9:CAP_1608_TDK, symbol Device:C
- added C15: 150pF, cappy7:G-188_MUR, symbol Device:C
- added C16, C17, C18, C19, C20: 22uF, cappy5:G-32_MUR, symbol Device:C
- added L1: 3.3uH, inducty1:IND_1050-WE-HCI_WRE, symbol Device:L
- added R43: 169kOhm, resisty169:RC0603N_YAG, symbol Device:R_US
- added R44: 36.1kOhm, resisty361:RESC1608X55N, symbol Device:R_US
- added R45: 52.3kOhm, resisty523:RC0603N_YAG, symbol Device:R_US
- added R46: 0, resisty0:RC0603N_VIS, symbol Device:R_US
- added R47: 100kOhm, resisty100:RES_CRCW_0603_VIS, symbol Device:R_US
- added R48: 10kOhm, resisty10:RC0603N_YAG, symbol Device:R_US
- added R49: 0, resisty0(2):RC0603N_YAG, symbol Device:R_US
- added R50: 49.9Ohm, resisty49:RC0603N_YAG, symbol Device:R_US
- added R51: 73.2kOhm, resisty732:RC0603N_YAG, symbol Device:R_US
- added U7: TPS56A37RPAR, bucky:RPA0010A-MFG, symbol TPS56A37RPAR:TPS56A37RPAR
Connections:
- new net: R43.2, R44.1, U7.1 (EN)
- new net: R49.1, R50.1, R51.1
- new net: R45.1, U7.10 (MODE)
- new net: C15.2, R48.1, R51.2, U7.2 (FB)
- new net: R47.1, U7.4 (PG)
- new net: C13.1, U7.5 (SS)
- new net: C14.2, L1.1, U7.6 (SW)
- new net: R46.1, U7.7 (BOOT)
- new net: C15.1, R49.2
- new net: C14.1, R46.2
- new net +24V: C10.1, C11.1, C12.1, R43.1, U7.8 (VIN)
- new net +5V: C16.1, C17.1, C18.1, C19.1, C20.2, L1.2, R47.2, R50.2
- new net AGND: C10.2, C11.2, C12.2, C13.2, C16.2, C17.2, C18.2, C19.2, C20.1, R44.2, R45.2, R48.2, U7.3 (AGND), U7.9 (PGND)

Commit message: 3.3v buck converter
Parts:
- added C36, C37: 10uF, cappy1:CAP_GRM32_3p5X2p7X2p7_MUR, symbol Device:C
- added C38, C40: 0.1uF, cappy3:CAP_885012206_WRE, symbol Device:C
- added C39: 47nF, cappy9:CAP_1608_TDK, symbol Device:C
- added C41: 150pF, cappy7:G-188_MUR, symbol Device:C
- added C42, C43, C44, C45, C46: 22uF, cappy5:G-32_MUR, symbol Device:C
- added L2: 2.2uH, inducty1:IND_1050-WE-HCI_WRE, symbol Device:L
- added R70: 169kOhm, resisty169:RC0603N_YAG, symbol Device:R_US
- added R71: 36.1kOhm, resisty361:RESC1608X55N, symbol Device:R_US
- added R72: 52.3kOhm, resisty523:RC0603N_YAG, symbol Device:R_US
- added R73: 0, resisty0:RC0603N_VIS, symbol Device:R_US
- added R74: 100kOhm, resisty100:RES_CRCW_0603_VIS, symbol Device:R_US
- added R75: 10kOhm, resisty10:RC0603N_YAG, symbol Device:R_US
- added R76: 0, resisty0(2):RC0603N_YAG, symbol Device:R_US
- added R77: 49.9Ohm, resisty49:RC0603N_YAG, symbol Device:R_US
- added R78: 45.3kOhm, resisty732:RC0603N_YAG, symbol Device:R_US
- added U14: TPS56A37RPAR, bucky:RPA0010A-MFG, symbol TPS56A37RPAR:TPS56A37RPAR
Connections:
- net +24V: now also C36.1, C37.1, C38.1, R70.1, U14.8 (VIN)
- net AGND: now also C36.2, C37.2, C38.2, C39.2, C42.2, C43.2, C44.2, C45.2, C46.1, R71.2, R72.2, R75.2, U14.3 (AGND), U14.9 (PGND)
- new net: R76.1, R77.1, R78.1
- new net: R70.2, R71.1, U14.1 (EN)
- new net: R72.1, U14.10 (MODE)
- new net: C41.2, R75.1, R78.2, U14.2 (FB)
- new net: R74.1, U14.4 (PG)
- new net: C39.1, U14.5 (SS)
- new net: C40.2, L2.1, U14.6 (SW)
- new net: R73.1, U14.7 (BOOT)
- new net: C40.1, R73.2
- new net: C41.1, R76.2
- new net +3.3V: C42.1, C43.1, C44.1, C45.1, C46.2, L2.2, R74.2, R77.2
Other:
- moved on the sheet: C10, C11, C12, C13, C14, C15, C16, C17, C18, C19, C20, L1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
