File: FlightComputerBoardV1/POWER.kicad_sch (KiCad schematic)
At the start: 152 parts, among them J19 RELAY_A1, J20 RELAY_A2, Q10 FDD4685, Q7 FDD4685, Q8 FDD4685, Q9 FDD4685, U14 TPS56A37RPAR, U15 LM74700, U16 INA260, U17 MCP9808_DFN, U18 LM74700, U21 PTPS2116DRLR, U22 TLV75533PDBVR, U23 LT4363IDE-2-PBF, U24 BSS138, U25 PS2811-1-F3-A, U26 PS2811-1-F3-A, U27 BSS138, U28 INA260, U29 MCP9808_DFN, U30 INA260, U31 MCP9808_DFN, U33 LTC4418IUF-TRPBF, U34 BAT46WJ_115, U35 BAT46WJ_115, U36 LT4363IDE-2-PBF, U7 TPS56A37RPAR

Commit message: The Calamity
Design Changes:
- Swapped actuators to run on H bridge circuit
- Added potentiometer feedback for actuators
- Assigned pins for actuator control
- Added gate driver circuits
Other:
- Created very preliminary BOM (lifesucks.csv)
- Assigned most footprints

To do:
- Standardize component naming
- Finalize BOM (screw terminals once physical design starts)
Parts:
- removed CR1, CR2: SMBJ26A, SMBJSeries_LTF, symbol SMBJ26A:SMBJ26A
- removed D11, D12: 1N4007, Diode_THT:D_DO-41_SOD81_P10.16mm_Horizontal, symbol Diode:1N4007
- removed J19: RELAY_A1, symbol Connector:Screw_Terminal_01x02
- removed J20: RELAY_A2, symbol Connector:Screw_Terminal_01x02
- removed MOSFET1, MOSFET2: NVMFS6H848NLT1G, DFN6_5X6_SO8FL_488AA_ONS, symbol NVMFS6H848NLT1G:NVMFS6H848NLT1G
- removed R58, R67: 100, RES_CRCW_0402, symbol FlightComputerBoardV1_Symbols:CRCW0402100RFKED
- removed R59, R68: 100k, RC0402N_PAN, symbol FlightComputerBoardV1_Symbols:ERJ-2GEJ104X
- removed R62, R64: 10k, symbol Device:R_US
- removed R63, R65: 670, symbol Device:R_US
- removed U15, U18: LM74700, Package_TO_SOT_SMD:SOT-23-6, symbol Power_Management:LM74700
- removed U24, U27: BSS138, SOT-23_3L_ONS, symbol FlightComputerBoardV1_Symbols:BSS138
- removed U25, U26: PS2811-1-F3-A, PS2811-1_REN, symbol PS2811_1_F3_A:PS2811-1-F3-A
- added C110, C111, C112, C113, C114, C115: 1uF, FlightComputerBoardV1_Footprints:CAP_GCM188_MUR, symbol Device:C
- added J22, J23: Screw_Terminal_01x05, Converter_DCDC:Converter_DCDC_Silvertel_Ag99xxLP_THT, symbol Connector:Screw_Terminal_01x05
- added M1, M2, M3, M4, M5, M6, M7, M8: CSD18532Q5B, FlightComputerBoardV1_Footprints:DNK8, symbol FlightComputerBoardV1_Symbols:CSD18532Q5B
- added R1, R58: R_Shunt, symbol Device:R_Shunt
- added R120, R121, R122, R124, R125, R126: 10k, Resistor_THT:R_Array_SIP4, symbol Device:R_US
- added R123, R127: 4.7k, Resistor_THT:R_Array_SIP4, symbol Device:R_US
- added R128, R129: 100, Resistor_THT:R_Array_SIP4, symbol Device:R_US
- added R130, R131: 1k, Resistor_THT:R_Array_SIP4, symbol Device:R_US
- added U15, U18: DRV8701ERGER, FlightComputerBoardV1_Footprints:RGE0024F, symbol FlightComputerBoardV1_Symbols:DRV8701ERGER
- C10, C11, C36, C37: footprint cappy1:CAP_GRM32_3p5X2p7X2p7_MUR -> FlightComputerBoardV1_Footprints:CAP_CL10_SAM
- C100, C102, C96, C97, C98: footprint UF_20_ADI -> FlightComputerBoardV1_Footprints:CAP_GCM15_MUR
- C101, C103: footprint UF_20_ADI -> FlightComputerBoardV1_Footprints:CAP_GRM0335_MUR
- C104, C99: footprint UF_20_ADI -> FlightComputerBoardV1_Footprints:G-155_MUR
- C105: footprint UF_20_ADI -> FlightComputerBoardV1_Footprints:CAP_CL10_SAM
- C106, C50, C51, C86, C87, C88, C90, C91, C92, C93: footprint (none) -> FlightComputerBoardV1_Footprints:CAP_GCM15_MUR
- C107, C108: footprint (none) -> FlightComputerBoardV1_Footprints:G-155_MUR
- C12, C14, C38, C40: footprint cappy3:CAP_885012206_WRE -> FlightComputerBoardV1_Footprints:CAP_GCM15_MUR
- C13, C39: footprint cappy9:CAP_1608_TDK -> FlightComputerBoardV1_Footprints:CAP_GCM15_MUR
- C15, C41: footprint cappy7:G-188_MUR -> FlightComputerBoardV1_Footprints:G-155_MUR_pF
- C16, C17, C18, C19, C20, C42, C43, C44, C45, C46: footprint cappy5:G-32_MUR -> FlightComputerBoardV1_Footprints:CAP_CL_05_SAM
- C47, C52: value 22nF -> 0.1u; footprint (none) -> FlightComputerBoardV1_Footprints:CAP_GCM15_MUR; now fitted
- C48: value 0.1uF -> 10uF; footprint (none) -> FlightComputerBoardV1_Footprints:CAP_CL10_SAM; now fitted
- C49: value 47uF -> 10uF; footprint (none) -> FlightComputerBoardV1_Footprints:CAP_CL10_SAM; now fitted
- C53: value 0.1uF -> 0.1u; footprint (none) -> FlightComputerBoardV1_Footprints:CAP_GCM15_MUR; now fitted
- C54: value 47uF -> 0.1u; footprint (none) -> FlightComputerBoardV1_Footprints:CAP_GCM15_MUR; now fitted
- C81, C82: footprint (none) -> FlightComputerBoardV1_Footprints:CAP_GCM188_MUR
- C83: footprint (none) -> FlightComputerBoardV1_Footprints:CAP_GRM31C_100u
- C84, C85: footprint DBV0005A_N -> FlightComputerBoardV1_Footprints:CAP_GCM188_MUR
- CR3, CR4: footprint SMASeries_LTF -> FlightComputerBoardV1_Footprints:SMASeries_LTF
- MOSFET3, MOSFET4: footprint D2PAK_SOT404_NEX -> FlightComputerBoardV1_Footprints:D2PAK_SOT404_NEX
- Q10, Q7, Q8, Q9: footprint TO252_FDD_ONS -> FlightComputerBoardV1_Footprints:TO252_FDD_ONS
- R113, R54, R55: footprint (none) -> FlightComputerBoardV1_Footprints:RC0805N_YAG
- R48: footprint resisty10:RC0603N_YAG -> FlightComputerBoardV1_Footprints:RC0805N_YAG
- U21: footprint DRL0008A-MFG -> (none)
- U22: footprint DBV0005A_N -> (none)
- U23, U36: footprint DFN-12_DE_LIT -> (none)
- U33: footprint UF_20_ADI -> (none)
- U34, U35: footprint SC-90_SOD323F_NEX -> (none)
Connections:
- net +24V: now also C48.1, C49.1, C110.1, C111.1, M1.5 (D), M1.6 (D), M1.7 (D), M1.8 (D), M3.5 (D), M3.6 (D), M3.7 (D), M3.8 (D), M5.5 (D), M5.6 (D), M5.7 (D), M5.8 (D), M7.5 (D), M7.6 (D), M7.7 (D), M7.8 (D), U15.1 (VM), U18.1 (VM)
- net +3.3V: now also R128.1, R129.1
- net AGND: now also C53.2, C54.2, C112.2, C113.1, C114.2, C115.1, J22.3 (Pin_3), J23.3 (Pin_3), R1.1, R123.1, R127.1, R58.1, U15.16 (GND), U15.20 (SN), U15.25 (PAD), U15.5 (GND), U18.16 (GND), U18.20 (SN), U18.25 (PAD), U18.5 (GND)
- net GND: no longer C47.2, C49.2, C52.2, C54.2
- net at C48.2: now also C110.2, U15.2 (VCP)
- net 24V_Unprotected renamed POT_LIN2
- net POT_LIN2: now also R131.1; no longer C49.1
- net Battery: no longer names the net of C52.1
- net Battery: now also U18.3 (CPH); no longer C53.1
- net Power Supply: no longer names the net of C47.1
- net Power Supply: now also U15.3 (CPH); no longer C48.1
- new net: R126.1, R127.2, U18.6 (VREF)
- new net: C115.2, R126.2, U18.7 (AVDD)
- new net: C47.2, U15.4 (CPL)
- new net: R122.1, R123.2, U15.6 (VREF)
- new net: C113.2, R122.2, U15.7 (AVDD)
- new net: C112.1, R120.2, R121.2, U15.8 (DVDD)
- new net: J23.2 (Pin_2), R129.2
- new net: C114.1, R124.2, R125.2, U18.8 (DVDD)
- new net: C111.2, C49.2, U18.2 (VCP)
- new net: C52.2, U18.4 (CPL)
- new net: J22.2 (Pin_2), R128.2
- new net: J22.4 (Pin_4), R131.2
- new net: J23.4 (Pin_4), R130.2
- new net FAULT_LIN1: R120.1, U15.9 (FAULT_N)
- new net FAULT_LIN2: R125.1, U18.9 (FAULT_N)
- new net GH1: M1.4 (G), M5.4 (G), U15.17 (GH1), U18.17 (GH1)
- new net GH2: M3.4 (G), M7.4 (G), U15.24 (GH2), U18.24 (GH2)
- new net GL1: M2.4 (G), M6.4 (G), U15.19 (GL1), U18.19 (GL1)
- new net GL2: M4.4 (G), M8.4 (G), U15.22 (GL2), U18.22 (GL2)
- new net IN1_LIN1: U15.15 (PH_IN1)
- new net IN1_LIN2: U18.15 (PH_IN1)
- new net IN2_LIN1: U15.14 (EN_IN2)
- new net IN2_LIN2: U18.14 (EN_IN2)
- new net POT_LIN1: C53.1, R130.1
- new net SH1: J22.1 (Pin_1), J23.1 (Pin_1), M1.1 (S), M1.2 (S), M1.3 (S), M2.5 (D), M2.6 (D), M2.7 (D), M2.8 (D), M5.1 (S), M5.2 (S), M5.3 (S), M6.5 (D), M6.6 (D), M6.7 (D), M6.8 (D), U15.18 (SH1), U18.18 (SH1)
- new net SH2: J22.5 (Pin_5), J23.5 (Pin_5), M3.1 (S), M3.2 (S), M3.3 (S), M4.5 (D), M4.6 (D), M4.7 (D), M4.8 (D), M7.1 (S), M7.2 (S), M7.3 (S), M8.5 (D), M8.6 (D), M8.7 (D), M8.8 (D), U15.23 (SH2), U18.23 (SH2)
- new net SLP_LIN1: U15.13 (SLEEP_N)
- new net SLP_LIN2: U18.13 (SLEEP_N)
- new net SN_LIN1: U15.10 (SNSOUT)
- new net SN_LIN2: R124.1, U18.10 (SNSOUT)
- new net SO_LIN1: U15.11 (SO)
- new net SO_LIN2: U18.11 (SO)
- new net SP: M2.1 (S), M2.2 (S), M2.3 (S), M4.1 (S), M4.2 (S), M4.3 (S), M6.1 (S), M6.2 (S), M6.3 (S), M8.1 (S), M8.2 (S), M8.3 (S), R1.4, R58.4, U15.21 (SP), U18.21 (SP)
- no-connect marks 19 -> 25
Other:
- note removed: "Feedback is for if we want absolute positioning feedback, will need extra pins and potentiomenter"
- note removed: "Replace with H bridge circuit, gate driver, and FETs"
- moved on the sheet: AC1, AC2
