File: FlightComputerBoardV1/MCU.kicad_sch (KiCad schematic)
At the start: 56 parts, among them J16 USB_C_Receptacle_USB2.0_16P, J17 Conn_ST_STDC14, J18 Micro_SD_Card, SW1 SW_Push, SW2 SW_Push, U20 STM32H723ZGTx, U32 USBLC6-2SC6, X1 32.768Khz, Y1 25Mhz

Commit message: Late night shenanigans
- Added radar module sheet
- Created symbols for: radar, RFD900xus
- Added RFD900xus
- Fixed PT voltage dividers
To do:
- Add decoupling and test points
- Finish finding appropriate gate driver for H bridge linear actuator circuit
Connections:
- net TX_UART_MC: now reaches U20.101 (PA9)
- net RX_UART_MC: now reaches U20.102 (PA10)
- net TX_UART_MC_R1: now reaches U20.85 (PD14)
- net RX_UART_MC_R1: now reaches U20.86 (PD15)
- net TX_UART_MC_R2: now reaches U20.96 (PC6)
- net RX_UART_MC_R2: now reaches U20.97 (PC7)

Commit message: The Calamity
Design Changes:
- Swapped actuators to run on H bridge circuit
- Added potentiometer feedback for actuators
- Assigned pins for actuator control
- Added gate driver circuits
Other:
- Created very preliminary BOM (lifesucks.csv)
- Assigned most footprints

To do:
- Standardize component naming
- Finalize BOM (screw terminals once physical design starts)
Parts:
- C57: footprint (none) -> FlightComputerBoardV1_Footprints:CAP_475MLHT_TAY
- C58, C59, C60, C61, C62, C63, C64, C65, C66, C67, C68, C71, C73, C78: footprint (none) -> FlightComputerBoardV1_Footprints:CAP_GCM15_MUR
- C69, C70, C72: footprint (none) -> FlightComputerBoardV1_Footprints:CAP_GCM188_MUR
- C74, C75: footprint (none) -> FlightComputerBoardV1_Footprints:CAP_GRT188R_MUR_22
- C76, C77: footprint XTAL_NX3215SA_NDK -> FlightComputerBoardV1_Footprints:G-155_MUR_91
- C79: footprint Capacitor_SMD:C_0402_1005Metric -> FlightComputerBoardV1_Footprints:CAP_GCM15_MUR
- C80: footprint Capacitor_SMD:C_0805_2012Metric -> FlightComputerBoardV1_Footprints:CAP_CL_05_SAM
- C94, C95: footprint XTAL_NX3215SA_NDK -> FlightComputerBoardV1_Footprints:G-155_MUR_10p
- R83: footprint Resistor_THT:R_Array_SIP4 -> FlightComputerBoardV1_Footprints:RC0805N_YAG
- R84: footprint (none) -> FlightComputerBoardV1_Footprints:RC0805N_YAG
- R91, R92, R93, R94: footprint (none) -> FlightComputerBoardV1_Footprints:RES_RC0805_YAG
- X1: footprint XTAL_NX3215SA_NDK -> (none)
Connections:
- net ADC1_INP2: now reaches U20.49 (PF11)
- net ADC1_INP6: now reaches U20.50 (PF12)
- net ADC2_INP2: now reaches U20.53 (PF13)
- net ADC2_INP6: now reaches U20.54 (PF14)
- net TIM1_CH1: now reaches U20.60 (PE9)
- net PE10_GPIO: now reaches U20.63 (PE10)
- net TIM1_CH2: now reaches U20.64 (PE11)
- net EXTI12: now reaches U20.65 (PE12)
- net TIM1_BKIN: now reaches U20.68 (PE15)
- net TIM8_BKIN: now reaches U20.87 (PG2)
- net PG5_GPIO: now reaches U20.90 (PG5)
- net EXTI16: now reaches U20.91 (PG6)
- net TIM8_CH3: now reaches U20.98 (PC8)
- net TIM8_CH4: now reaches U20.99 (PC9)
