File: FlightComputerBoardV1/Peripherals-IMU.kicad_sch (KiCad schematic)
At the start: 39 parts, among them U10 LSM6DSOXTR, U11 LIS3MDLTR, U12 LIS3MDLTR, U13 LIS3MDLTR, U8 LSM6DSOXTR, U9 LSM6DSOXTR

Commit message: Test Points, BMP581
- Added I2C and other test points to schematic
- Added BMP581 symbol, footprint, and schematic on Peripherals sheet
Parts:
- added C55, C56: 100nF, LSM6DSOXTR:PQFN50P250X300X86-14N, symbol Device:C
- added R79, R80: 10k, symbol Device:R_US
- added TP10, TP11, TP12, TP13, TP14, TP15, TP16, TP5, TP6, TP7, TP8, TP9: TestPoint, symbol Connector:TestPoint
- added U19: BMP581, FlightComputerBoardV1_Footprints:BMP581_QFN10, symbol FlightComputerBoardV1_Symbols:BMP581
Connections:
- net +3.3V: now also C55.1, C56.1, R79.1, R80.1, U19.1 (VDDIO), U19.10 (VDD), U19.5 (SDO), U19.6 (CSB)
- net GND: now also C55.2, C56.2, U19.3 (VSS), U19.8 (VSS), U19.9 (VSS)
- net SCL_I2C_X: now also TP13.1, TP15.1, TP7.1, TP9.1
- net SCL_I2C_Y: now also TP11.1, TP5.1
- net SDA_I2C_X: now also TP10.1, TP14.1, TP16.1, TP8.1
- net SDA_I2C_Y: now also TP12.1, TP6.1
- new net SCL_I2C_A: R79.2, U19.2 (SCK)
- new net SDA_I2C_A: R80.2, U19.4 (SDI)
- no-connect marks 18 -> 19
Other:
- note added: "BMP581 - I2C"
- note added: "I2C ADDRESS: 0X47 I2C BUS: TBD"
- moved on the sheet: C23, C24, C27, C28, C29, C30, C31, C32, C33, C34, C35, R55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

Commit message: Addition to MCU sheet and peripheral connection complete
Parts:
- R53, R54, R55, R56, R58, R59, R62, R63, R64, R65, R67, R68, R79, R80: value 10k -> 4.7k
Connections:
- net SCL_I2C_X is gone; now on net SCL_I2C_1: R53.2, R55.2, R62.2, R64.2, TP13.1, TP15.1, TP7.1, TP9.1, U11.1 (SCL/SPC), U12.1 (SCL/SPC), U8.13 (SCL), U9.13 (SCL)
- net SDA_I2C_X is gone; now on net SDA_I2C_1: R54.2, R56.2, R63.2, R65.2, TP10.1, TP14.1, TP16.1, TP8.1, U11.11 (SDA/SDI/SDO), U12.11 (SDA/SDI/SDO), U8.14 (SDA), U9.14 (SDA)
- net SCL_I2C_A renamed SCL_I2C_1
- net SCL_I2C_Y renamed SCL_I2C_2
- net SDA_I2C_A renamed SDA_I2C_1
- net SDA_I2C_Y renamed SDA_I2C_2
Other:
- note added: "I2C ADDRESS: 0X1C I2C BUS: 1"
- note added: "I2C ADDRESS: 0X1C I2C BUS: 2"
- note added: "I2C ADDRESS: 0X1E I2C BUS: 1"
- note added: "I2C ADDRESS: 0X47 I2C BUS: 1"
- note added: "I2C ADDRESS: 0X6A I2C BUS: 1"
- note added: "I2C ADDRESS: 0X6A I2C BUS: 2"
- note added: "I2C ADDRESS: 0X6B I2C BUS: 1"
- note removed: "I2C ADDRESS: 0X1C I2C BUS: TBD"
- note removed: "I2C ADDRESS: 0X1E I2C BUS: TBD"
- note removed: "I2C ADDRESS: 0X47 I2C BUS: TBD"
- note removed: "I2C ADDRESS: 0X6A I2C BUS: TBD"
- note removed: "I2C ADDRESS: 0X6B I2C BUS: TBD"
Changed lines of the file:
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@@
 		)
 	)
-	(text "I2C ADDRESS: 0X1C\nI2C BUS: TBD"
+	(text "I2C ADDRESS: 0X1C\nI2C BUS: 1\n"
 		(exclude_from_sim no)
 		(at 117.856 148.336 0)
@@
 		)
 	)
-	(text "I2C ADDRESS: 0X6A\nI2C BUS: TBD"
+	(text "I2C ADDRESS: 0X6A\nI2C BUS: 1\n"
 		(exclude_from_sim no)
 		(at 130.048 26.67 0)
@@
 		)
 	)
-	(text "I2C ADDRESS: 0X6A\nI2C BUS: TBD"
+	(text "I2C ADDRESS: 0X6A\nI2C BUS: 2\n"
 		(exclude_from_sim no)
 		(at 185.928 78.74 0)
@@
 		)
 	)
-	(text "I2C ADDRESS: 0X6B\nI2C BUS: TBD"
+	(text "I2C ADDRESS: 0X6B\nI2C BUS: 1\n"
 		(exclude_from_sim no)
 		(at 263.398 26.67 0)
@@
 		)
 	)
-	(text "I2C ADDRESS: 0X47\nI2C BUS: TBD"
+	(text "I2C ADDRESS: 0X47\nI2C BUS: 1"
 		(exclude_from_sim no)
 		(at 357.124 172.72 0)
@@
 		)
 	)
-	(text "I2C ADDRESS: 0X1C\nI2C BUS: TBD"
+	(text "I2C ADDRESS: 0X1C\nI2C BUS: 2\n"
 		(exclude_from_sim no)
 		(at 161.036 205.486 0)
@@
 		)
 	)
-	(text "I2C ADDRESS: 0X1E\nI2C BUS: TBD"
+	(text "I2C ADDRESS: 0X1E\nI2C BUS: 1\n"
 		(exclude_from_sim no)
 		(at 216.916 148.336 0)
@@
 		)
 	)
-	(hierarchical_label "SDA_I2C_X"
+	(hierarchical_label "SDA_I2C_1"
 		(shape bidirectional)
 		(at 67.31 50.8 180)
@@
 		)
 	)
-	(hierarchical_label "SCL_I2C_X"
+	(hierarchical_label "SCL_I2C_1"
 		(shape bidirectional)
 		(at 194.31 48.26 180)
@@
 		)
 	)
-	(hierarchical_label "SCL_I2C_X"
+	(hierarchical_label "SCL_I2C_1"
 		(shape bidirectional)
 		(at 67.31 48.26 180)
@@
 		)
 	)
-	(hierarchical_label "SDA_I2C_Y"
+	(hierarchical_label "SDA_I2C_2"
 		(shape bidirectional)
 		(at 91.44 234.95 180)
@@
 		)
 	)
-	(hierarchical_label "SDA_I2C_X"
+	(hierarchical_label "SDA_I2C_1"
 		(shape bidirectional)
 		(at 154.94 177.8 180)
@@
 		)
 	)
-	(hierarchical_label "SCL_I2C_Y"
+	(hierarchical_label "SCL_I2C_2"
 		(shape bidirectional)
 		(at 116.84 100.33 180)
@@
 		)
 	)
-	(hierarchical_label "SDA_I2C_Y"
+	(hierarchical_label "SDA_I2C_2"
 		(shape bidirectional)
 		(at 116.84 102.87 180)
@@
 		)
 	)
-	(hierarchical_label "SCL_I2C_X"
+	(hierarchical_label "SCL_I2C_1"
 		(shape bidirectional)
 		(at 154.94 175.26 180)
@@
 		)
 	)
-	(hierarchical_label "SCL_I2C_A"
-		(shape input)
+	(hierarchical_label "SCL_I2C_1"
+		(shape bidirectional)
 		(at 314.96 195.58 180)
 		(effects
@@
 		)
 	)
-	(hierarchical_label "SDA_I2C_X"
+	(hierarchical_label "SDA_I2C_1"
 		(shape bidirectional)
 		(at 194.31 50.8 180)
@@
 		)
 	)
-	(hierarchical_label "SDA_I2C_A"
-		(shape input)
+	(hierarchical_label "SDA_I2C_1"
+		(shape bidirectional)
 		(at 323.85 205.74 180)
 		(effects
@@
 		)
 	)
-	(hierarchical_label "SCL_I2C_Y"
+	(hierarchical_label "SCL_I2C_2"
 		(shape bidirectional)
 		(at 91.44 232.41 180)
@@
 		)
 	)
-	(hierarchical_label "SCL_I2C_X"
+	(hierarchical_label "SCL_I2C_1"
 		(shape bidirectional)
 		(at 50.8 175.26 180)
@@
 		)
 	)
-	(hierarchical_label "SDA_I2C_X"
+	(hierarchical_label "SDA_I2C_1"
 		(shape bidirectional)
 		(at 50.8 177.8 180)
@@
 			)
 		)
-		(property "Value" "10k"
+		(property "Value" "4.7k"
 			(at 152.654 95.25 0)
 			(show_name no)
@@
 			)
 		)
-		(property "Value" "10k"
+		(property "Value" "4.7k"
 			(at 326.644 186.69 0)
 			(show_name no)
@@
 			)
 		)
-		(property "Value" "10k"
+		(property "Value" "4.7k"
 			(at 104.648 42.926 0)
 			(show_name no)
@@
 			)
 		)
-		(property "Value" "10k"
+		(property "Value" "4.7k"
 			(at 230.124 43.18 0)
 			(show_name no)
@@
 			)
 		)
-		(property "Value" "10k"
+		(property "Value" "4.7k"
 			(at 160.528 94.996 0)
 			(show_name no)
@@
 			)
 		)
-		(property "Value" "10k"
+		(property "Value" "4.7k"
 			(at 317.754 186.69 0)
 			(show_name no)
@@
 			)
 		)
-		(property "Value" "10k"
+		(property "Value" "4.7k"
 			(at 136.144 228.6 0)
 			(show_name no)
@@
 			)
 		)
-		(property "Value" "10k"
+		(property "Value" "4.7k"
 			(at 185.674 171.45 0)
 			(show_name no)
@@
 			)
 		)
-		(property "Value" "10k"
+		(property "Value" "4.7k"
 			(at 192.024 171.45 0)
 			(show_name no)
@@
 			)
 		)
-		(property "Value" "10k"
+		(property "Value" "4.7k"
 			(at 92.964 171.45 0)
 			(show_name no)
@@
 			)
 		)
-		(property "Value" "10k"
+		(property "Value" "4.7k"
 			(at 237.998 42.926 0)
 			(show_name no)
@@
 			)
 		)
-		(property "Value" "10k"
+		(property "Value" "4.7k"
 			(at 86.614 171.45 0)
 			(show_name no)
@@
 			)
 		)
-		(property "Value" "10k"
+		(property "Value" "4.7k"
 			(at 96.774 43.18 0)
 			(show_name no)
@@
 			)
 		)
-		(property "Value" "10k"
+		(property "Value" "4.7k"
 			(at 129.794 228.6 0)
 			(show_name no)

Commit message: Fixed I2C pull ups
Parts:
- removed R53, R54, R55, R56, R58, R59, R62, R63, R64, R65, R67, R68, R79, R80: 4.7k, symbol Device:R_US
Other:
- moved on the sheet: TP5, TP6, TP7, TP8

Commit message: The Calamity
Design Changes:
- Swapped actuators to run on H bridge circuit
- Added potentiometer feedback for actuators
- Assigned pins for actuator control
- Added gate driver circuits
Other:
- Created very preliminary BOM (lifesucks.csv)
- Assigned most footprints

To do:
- Standardize component naming
- Finalize BOM (screw terminals once physical design starts)
Parts:
- C21, C22, C23, C24, C25, C26, C27, C28, C30, C31, C33, C34, C55, C56: footprint LSM6DSOXTR:PQFN50P250X300X86-14N -> FlightComputerBoardV1_Footprints:CAP_GCM15_MUR
- C29, C32, C35: footprint LSM6DSOXTR:PQFN50P250X300X86-14N -> FlightComputerBoardV1_Footprints:CAP_GCM188_MUR
- R52, R57, R60, R61, R66, R69: footprint (none) -> FlightComputerBoardV1_Footprints:RES_RC0805_YAG
Changed lines of the file:
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@@
 			)
 		)
-		(property "Footprint" "LSM6DSOXTR:PQFN50P250X300X86-14N"
+		(property "Footprint" "FlightComputerBoardV1_Footprints:CAP_GCM188_MUR"
 			(at 153.3652 165.1 0)
 			(hide yes)
@@
 			)
 		)
-		(property "Footprint" ""
+		(property "Footprint" "FlightComputerBoardV1_Footprints:RES_RC0805_YAG"
 			(at 199.136 166.624 90)
 			(hide yes)
@@
 			)
 		)
-		(property "Footprint" "LSM6DSOXTR:PQFN50P250X300X86-14N"
+		(property "Footprint" "FlightComputerBoardV1_Footprints:CAP_GCM15_MUR"
 			(at 185.1152 222.25 0)
 			(hide yes)
@@
 			)
 		)
-		(property "Footprint" ""
+		(property "Footprint" "FlightComputerBoardV1_Footprints:RES_RC0805_YAG"
 			(at 167.386 94.234 90)
 			(hide yes)
@@
 			)
 		)
-		(property "Footprint" "LSM6DSOXTR:PQFN50P250X300X86-14N"
+		(property "Footprint" "FlightComputerBoardV1_Footprints:CAP_GCM15_MUR"
 			(at 307.0352 45.72 0)
 			(hide yes)
@@
 			)
 		)
-		(property "Footprint" "LSM6DSOXTR:PQFN50P250X300X86-14N"
+		(property "Footprint" "FlightComputerBoardV1_Footprints:CAP_GCM15_MUR"
 			(at 291.7952 199.39 0)
 			(hide yes)
@@
 			)
 		)
-		(property "Footprint" "LSM6DSOXTR:PQFN50P250X300X86-14N"
+		(property "Footprint" "FlightComputerBoardV1_Footprints:CAP_GCM15_MUR"
 			(at 293.0652 45.72 0)
 			(hide yes)
@@
 			)
 		)
-		(property "Footprint" "LSM6DSOXTR:PQFN50P250X300X86-14N"
+		(property "Footprint" "FlightComputerBoardV1_Footprints:CAP_GCM15_MUR"
 			(at 94.9452 194.31 0)
 			(hide yes)
@@
 			)
 		)
-		(property "Footprint" "LSM6DSOXTR:PQFN50P250X300X86-14N"
+		(property "Footprint" "FlightComputerBoardV1_Footprints:CAP_GCM15_MUR"
 			(at 138.1252 251.46 0)
 			(hide yes)
@@
 			)
 		)
-		(property "Footprint" ""
+		(property "Footprint" "FlightComputerBoardV1_Footprints:RES_RC0805_YAG"
 			(at 143.256 223.774 90)
 			(hide yes)
@@
 			)
 		)
-		(property "Footprint" "LSM6DSOXTR:PQFN50P250X300X86-14N"
+		(property "Footprint" "FlightComputerBoardV1_Footprints:CAP_GCM15_MUR"
 			(at 194.0052 194.31 0)
 			(hide yes)
@@
 			)
 		)
-		(property "Footprint" "LSM6DSOXTR:PQFN50P250X300X86-14N"
+		(property "Footprint" "FlightComputerBoardV1_Footprints:CAP_GCM15_MUR"
 			(at 215.5952 97.79 0)
 			(hide yes)
@@
 			)
 		)
-		(property "Footprint" "LSM6DSOXTR:PQFN50P250X300X86-14N"
+		(property "Footprint" "FlightComputerBoardV1_Footprints:CAP_GCM188_MUR"
 			(at 252.4252 165.1 0)
 			(hide yes)
@@
 			)
 		)
-		(property "Footprint" "LSM6DSOXTR:PQFN50P250X300X86-14N"
+		(property "Footprint" "FlightComputerBoardV1_Footprints:CAP_GCM15_MUR"
 			(at 393.3952 198.12 0)
 			(hide yes)
@@
 			)
 		)
-		(property "Footprint" ""
+		(property "Footprint" "FlightComputerBoardV1_Footprints:RES_RC0805_YAG"
 			(at 244.856 42.164 90)
 			(hide yes)
@@
 			)
 		)
-		(property "Footprint" "LSM6DSOXTR:PQFN50P250X300X86-14N"
+		(property "Footprint" "FlightComputerBoardV1_Footprints:CAP_GCM15_MUR"
 			(at 240.9952 165.1 0)
 			(hide yes)
@@
 			)
 		)
-		(property "Footprint" "LSM6DSOXTR:PQFN50P250X300X86-14N"
+		(property "Footprint" "FlightComputerBoardV1_Footprints:CAP_GCM188_MUR"
 			(at 196.5452 222.25 0)
 			(hide yes)
@@
 			)
 		)
-		(property "Footprint" ""
+		(property "Footprint" "FlightComputerBoardV1_Footprints:RES_RC0805_YAG"
 			(at 111.506 42.164 90)
 			(hide yes)
@@
 			)
 		)
-		(property "Footprint" "LSM6DSOXTR:PQFN50P250X300X86-14N"
+		(property "Footprint" "FlightComputerBoardV1_Footprints:CAP_GCM15_MUR"
 			(at 159.7152 45.72 0)
 			(hide yes)
@@
 			)
 		)
-		(property "Footprint" "LSM6DSOXTR:PQFN50P250X300X86-14N"
+		(property "Footprint" "FlightComputerBoardV1_Footprints:CAP_GCM15_MUR"
 			(at 141.9352 165.1 0)
 			(hide yes)
@@
 			)
 		)
-		(property "Footprint" "LSM6DSOXTR:PQFN50P250X300X86-14N"
+		(property "Footprint" "FlightComputerBoardV1_Footprints:CAP_GCM15_MUR"
 			(at 173.6852 45.72 0)
 			(hide yes)
@@
 			)
 		)
-		(property "Footprint" "LSM6DSOXTR:PQFN50P250X300X86-14N"
+		(property "Footprint" "FlightComputerBoardV1_Footprints:CAP_GCM15_MUR"
 			(at 229.5652 97.79 0)
 			(hide yes)
@@
 			)
 		)
-		(property "Footprint" ""
+		(property "Footprint" "FlightComputerBoardV1_Footprints:RES_RC0805_YAG"
 			(at 100.076 166.624 90)
 			(hide yes)
