File: FlightComputerBoardV1/RADAR.kicad_sch (KiCad schematic)
At the start: 6 parts

Commit message: The Calamity
Design Changes:
- Swapped actuators to run on H bridge circuit
- Added potentiometer feedback for actuators
- Assigned pins for actuator control
- Added gate driver circuits
Other:
- Created very preliminary BOM (lifesucks.csv)
- Assigned most footprints

To do:
- Standardize component naming
- Finalize BOM (screw terminals once physical design starts)
Parts:
- RAD1, RAD2: footprint RC0402N_PAN -> (none)
Changed lines of the file:
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@@
 			)
 		)
-		(property "Footprint" "RC0402N_PAN"
+		(property "Footprint" ""
 			(at 63.5 111.76 0)
 			(hide yes)
@@
 			)
 		)
-		(property "Footprint" "RC0402N_PAN"
+		(property "Footprint" ""
 			(at 63.5 147.32 0)
 			(hide yes)
